File: ESP_Scale/PCB/ESP_Weight_Main/ESP_Weight.kicad_pcb (KiCad board)
At the start: 4 copper layers, 116.5 x 53 mm, 112 parts, among them J1 VIN, J2 RS232, J3 Motor, J4 Comm, J5 SD_Memory, J6 PWR_SW, J7 RS232, J8 RTC_BAT, J9 DEBUG, K1 PWR_RELAY, Q1 BS250, SW1 RST, U1 H7150-1, U10 ISO1540, U11 ADuM1402xRW, U12 EL817, U13 MAX232, U14 P82B715DR, U15 SRV05-4, U16 PCF8563T, U2 DRV8871DDA, U3 EL817, U4 B1203S-1WR3, U5 ESP32-WROOM-32U, U6 B1205S-1WR3, U7 EL817, U8 TPD2E007, U9 TPD2E007, Y1 32.768

Commit message: PCB File 업데이트
Parts:
- removed Q1: BS250, Package_TO_SOT_SMD:SOT-23
- removed R18: 10k, Resistor_SMD:R_0603_1608Metric
- removed RN1: 10k, Resistor_SMD:R_Cat16-4
- H1, H2, H3, H4: footprint MountingHole:MountingHole_3.2mm_M3 -> MountingHole:MountingHole_3.2mm_M3_Pad
- JP1, JP2: footprint Jumper:SolderJumper-2_P1.3_THT -> KIcad:SolderJumper-2_P1.3_THT
Connections:
- C27 pad 1: Net-(J5-VDD) -> +3.3V
- J5 pad 4: Net-(J5-VDD) -> +3.3V
- U5 pad 9: /SD_PWR -> unconnected-(U5-IO33-Pad9)
Routing:
- net /SD_PWR: track 26.3 -> 0.00 mm, vias 2 -> 0
- net Net-(J5-VDD): track 19.8 -> 0.00 mm, vias 2 -> 0
- net +3.3V: track 35.1 -> 47.1 mm, vias 11 -> 13
- net /SD_MOSI: track 42.3 -> 37.3 mm
- net /SD_MISO: track 36.0 -> 31.7 mm
- net /SD_CLK: track 33.1 -> 29.4 mm
- net /SD_CS: track 30.5 -> 27.5 mm
- net /IO0: track 51.3 -> 52.0 mm
- net GNDPWR: vias 187 -> 177
- net GND: vias 196 -> 187
- net /Communication/5V_Comm_GND: vias 116 -> 115
Other:
- board text added: "FishingScale_MainBoard_V3.7"
- board text removed: "FishingScale_MainBoard_V3.6"
