File: ESP_Scale/PCB/ESP_Weight_Main/ESP_Weight.kicad_sch (KiCad schematic)
At the start: 34 parts, among them J5 SD_Memory, J8 RTC_BAT, J9 DEBUG, Q1 BS250, SW1 RST, U16 PCF8563T, U5 ESP32-WROOM-32U, Y1 32.768

Commit message: PCB File 업데이트
Parts:
- removed Q1: BS250, Package_TO_SOT_SMD:SOT-23, symbol Transistor_FET:AO3401A
- removed R18: 10k, Resistor_SMD:R_0603_1608Metric, symbol Device:R_Small_US
- removed RN1: 10k, Resistor_SMD:R_Cat16-4, symbol Device:R_Pack04
- H1, H2, H3, H4: footprint MountingHole:MountingHole_3.2mm_M3 -> MountingHole:MountingHole_3.2mm_M3_Pad
- JP1, JP2: footprint Jumper:SolderJumper-2_P1.3_THT -> KIcad:SolderJumper-2_P1.3_THT
Connections:
- net +3.3V: now also C27.1, J5.4 (VDD)
- net SD_PWR: no longer names the net of U5.9 (IO33)
