File: ESP_Scale/PCB/ESP_Weight_Panel/Panel_board.kicad_pcb (KiCad board)
At the start: 4 copper layers, 46.5 x 130.4 mm, 94 parts, among them J1 LED_12V, J10 BTN4, J11 Comm, J12 RFID_Module, J2 Loadcell, J3 LCD_1602, J5 NET, J6 TARE, J7 BTN1, J8 BTN2, J9 BTN3, Q2 FDC655BN, U1 B1205S-1WR3, U10 TPD2E007, U11 ULN2003, U2 ISO1540, U3 EL817, U4 NAU7802, U5 MCP23017_ML, U6 EL817, U7 P82B715DR, U8 B1205S-1WR3, U9 SRV05-4

Commit message: PCB File 업데이트
Parts:
- removed G***: LOGO, KIcad:FishingScale
- H1, H2: footprint MountingHole:MountingHole_3.2mm_M3 -> MountingHole:MountingHole_3.2mm_M3_Pad
- moved BZ1 7.78 mm to (12.8, 17.8), turned to -90 degrees
- turned D3 to -90 degrees
Connections:
- BZ1 pad 1: Net-(BZ1--) -> +5V
- BZ1 pad 2: GND -> Net-(BZ1-+)
- D3 pad 1: Net-(BZ1--) -> +5V
- D3 pad 2: GND -> Net-(BZ1-+)
- U11 pad 10: Net-(BZ1--) -> Net-(BZ1-+)
- U5 pad 21: /BTN3 -> unconnected-(U5-GPA4-Pad21)
- U5 pad 22: /BTN4 -> /BTN3
- U5 pad 23: unconnected-(U5-GPA6-Pad23) -> /BTN4
Routing:
- net Net-(BZ1--): track 67.3 -> 0.00 mm
- net Net-(BZ1-+): track 0.00 -> 67.3 mm
- net +5V: track 31.5 -> 40.4 mm
- net /BTN3: track 9.38 -> 8.31 mm
- net /BTN4: track 16.7 -> 16.2 mm
- net GND: vias 11 -> 10
Other:
- board size 46.5 x 130.4 mm -> 46.5 x 131 mm
- board text added: "FishingScale_PanelBoard V3.5"
- board text removed: "FishingScale_PanelBoard_V3.4"
