File: ESP_Scale/PCB/ESP_Weight_Panel/Panel_board.kicad_sch (KiCad schematic)
At the start: 42 parts, among them J10 BTN4, J2 Loadcell, J3 LCD_1602, J5 NET, J6 TARE, J7 BTN1, J8 BTN2, J9 BTN3, U11 ULN2003, U4 NAU7802, U5 MCP23017_ML

Commit message: PCB File 업데이트
Parts:
- H1, H2: footprint MountingHole:MountingHole_3.2mm_M3 -> MountingHole:MountingHole_3.2mm_M3_Pad
Connections:
- net +5V: now also BZ1.1 (-), D3.1 (K)
- net BTN3: now also U5.22 (GPA5); no longer U5.21 (GPA4)
- net BTN4: now also U5.23 (GPA6); no longer U5.22 (GPA5)
- net GND: no longer BZ1.2 (+), D3.2 (A)
- new net: BZ1.2 (+), D3.2 (A), U11.10 (O7)
- no-connect marks 0 -> 1
Other:
- moved on the sheet: BZ1
Changed lines of the file:
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@@
   (junction (at 198.12 109.22) (diameter 0) (color 0 0 0 0)
   )
+  (junction (at 66.04 149.86) (diameter 0) (color 0 0 0 0)
+  )
+  (junction (at 113.03 69.85) (diameter 0) (color 0 0 0 0)
+  )
+  (junction (at 247.65 149.86) (diameter 0) (color 0 0 0 0)
+  )
+  (junction (at 121.92 160.02) (diameter 0) (color 0 0 0 0)
+  )
+  (junction (at 247.65 128.27) (diameter 0) (color 0 0 0 0)
+  )
+  (junction (at 180.34 88.9) (diameter 0) (color 0 0 0 0)
+  )
+  (junction (at 247.65 85.09) (diameter 0) (color 0 0 0 0)
+  )
   (junction (at 205.74 109.22) (diameter 0) (color 0 0 0 0)
   )
-  (junction (at 66.04 149.86) (diameter 0) (color 0 0 0 0)
-  )
-  (junction (at 113.03 69.85) (diameter 0) (color 0 0 0 0)
-  )
-  (junction (at 247.65 149.86) (diameter 0) (color 0 0 0 0)
-  )
-  (junction (at 121.92 160.02) (diameter 0) (color 0 0 0 0)
-  )
-  (junction (at 247.65 128.27) (diameter 0) (color 0 0 0 0)
-  )
-  (junction (at 180.34 88.9) (diameter 0) (color 0 0 0 0)
-  )
-  (junction (at 247.65 85.09) (diameter 0) (color 0 0 0 0)
-  )
   (junction (at 95.25 115.57) (diameter 0) (color 0 0 0 0)
   )
@@
   (junction (at 62.23 158.75) (diameter 0) (color 0 0 0 0)
   )
+  (no_connect (at 130.81 110.49))
   (wire (pts (xy 53.34 158.75) (xy 62.23 158.75))
     (stroke (width 0) (type default))
@@
     (effects (font (size 1.27 1.27)) (justify right bottom))
   )
-  (label "BTN4" (at 130.81 113.03 0) (fields_autoplaced)
+  (label "BTN4" (at 130.81 115.57 0) (fields_autoplaced)
     (effects (font (size 1.27 1.27)) (justify left bottom))
   )
@@
     (effects (font (size 1.27 1.27)) (justify right bottom))
   )
-  (label "BTN3" (at 130.81 110.49 0) (fields_autoplaced)
+  (label "BTN3" (at 130.81 113.03 0) (fields_autoplaced)
     (effects (font (size 1.27 1.27)) (justify left bottom))
   )
@@
     )
   )
-  (symbol (lib_id "Diode:1N4148") (at 201.93 109.22 0) (unit 1)
-    (in_bom yes) (on_board yes) (dnp no)
-    (property "Reference" "D3" (at 200.66 111.76 0)
-      (effects (font (size 1.27 1.27)) (justify left))
-    )
-    (property "Value" "1N4148" (at 198.12 114.3 0)
+  (symbol (lib_id "Diode:1N4148") (at 201.93 109.22 0) (mirror y) (unit 1)
+    (in_bom yes) (on_board yes) (dnp no)
+    (property "Reference" "D3" (at 203.2 111.76 0)
+      (effects (font (size 1.27 1.27)) (justify left))
+    )
+    (property "Value" "1N4148" (at 205.74 114.3 0)
       (effects (font (size 1.27 1.27)) (justify left))
     )
@@
     )
   )
-  (symbol (lib_id "Panel_board-rescue:Buzzer-Device") (at 201.93 101.6 90) (unit 1)
-    (in_bom yes) (on_board yes) (dnp no)
-    (property "Reference" "BZ1" (at 198.12 99.06 90)
-      (effects (font (size 1.27 1.27)) (justify left))
-    )
-    (property "Value" "Buzzer" (at 198.12 101.6 90)
-      (effects (font (size 1.27 1.27)) (justify left))
-    )
-    (property "Footprint" "Buzzer_Beeper:Buzzer_12x9.5RM7.6" (at 199.39 102.235 90)
-      (effects (font (size 1.27 1.27)) hide)
-    )
-    (property "Datasheet" "~" (at 199.39 102.235 90)
+  (symbol (lib_id "Panel_board-rescue:Buzzer-Device") (at 201.93 101.6 270) (mirror x) (unit 1)
+    (in_bom yes) (on_board yes) (dnp no)
+    (property "Reference" "BZ1" (at 205.74 99.06 90)
+      (effects (font (size 1.27 1.27)) (justify left))
+    )
+    (property "Value" "Buzzer" (at 205.74 101.6 90)
+      (effects (font (size 1.27 1.27)) (justify left))
+    )
+    (property "Footprint" "Buzzer_Beeper:Buzzer_12x9.5RM7.6" (at 204.47 102.235 90)
+      (effects (font (size 1.27 1.27)) hide)
+    )
+    (property "Datasheet" "~" (at 204.47 102.235 90)
       (effects (font (size 1.27 1.27)) hide)
     )
@@
       (effects (font (size 1.27 1.27)) (justify left))
     )
-    (property "Footprint" "MountingHole:MountingHole_3.2mm_M3" (at 148.59 176.53 0)
+    (property "Footprint" "MountingHole:MountingHole_3.2mm_M3_Pad" (at 148.59 176.53 0)
       (effects (font (size 1.27 1.27)) hide)
     )
@@
       (effects (font (size 1.27 1.27)) (justify left))
     )
-    (property "Footprint" "MountingHole:MountingHole_3.2mm_M3" (at 148.59 170.18 0)
+    (property "Footprint" "MountingHole:MountingHole_3.2mm_M3_Pad" (at 148.59 170.18 0)
       (effects (font (size 1.27 1.27)) hide)
     )
@@
     )
   )
-  (symbol (lib_id "power:GND") (at 205.74 109.22 90) (unit 1)
-    (in_bom yes) (on_board yes) (dnp no) (fields_autoplaced)
-    (property "Reference" "#PWR02" (at 212.09 109.22 0)
-      (effects (font (size 1.27 1.27)) hide)
-    )
-    (property "Value" "GND" (at 209.55 109.22 90)
-      (effects (font (size 1.27 1.27)) (justify right))
+  (symbol (lib_id "power:+5V") (at 205.74 109.22 270) (unit 1)
+    (in_bom yes) (on_board yes) (dnp no)
+    (property "Reference" "#PWR02" (at 201.93 109.22 0)
+      (effects (font (size 1.27 1.27)) hide)
+    )
+    (property "Value" "+5V" (at 210.1342 109.601 0)
+      (effects (font (size 1.27 1.27)))
     )
     (property "Footprint" "" (at 205.74 109.22 0)
